File: usb-b2c.kicad_pcb (KiCad board)
At the start: 2 copper layers, 15 x 12 mm, 4 parts, among them J1 USB_B, J2 USB_C_Receptacle_USB2.0

Commit message: prepare for manufacturing
Other:
- board size 15 x 12 mm -> 15 x 17 mm
